Commit message: 更换 mujoco_ros2_control

File: src/fr3_sim/urdf/fr3.urdf.xacro (robot description, xacro)
@@ -24,23 +24,24 @@
     <ros2_control name="MujocoSystem" type="system">
         <hardware>
-            <plugin>mujoco_ros2_control/MujocoSystem</plugin>
+            <plugin>mujoco_ros2_control/MujocoSystemInterface</plugin>
+            <param name="mujoco_model">$(find fr3_sim)/config/fr3_mujoco.xml</param>
+            <param name="pids_config_file">$(find fr3_sim)/config/pid_gains.yaml</param>
         </hardware>
-        <xacro:macro name="configure_joint" params="name">
+        <xacro:macro name="configure_joint" params="name ip:=0">
             <joint name="${name}">
                 <command_interface name="position"/>
-                <command_interface name="velocity"/>
-                <command_interface name="effort"/>
-                <state_interface name="position"/>
+                <!-- <command_interface name="velocity"/>
+                <command_interface name="effort"/> -->
+                <state_interface name="position">
+                    <param name="initial_value">${ip}</param>
+                </state_interface>
                 <state_interface name="velocity"/>
                 <state_interface name="effort"/>
             </joint>
         </xacro:macro>
-        <xacro:configure_joint name="fr3_joint1"/>
-        <xacro:configure_joint name="fr3_joint2"/>
-        <xacro:configure_joint name="fr3_joint3"/>
-        <xacro:configure_joint name="fr3_joint4"/>
-        <xacro:configure_joint name="fr3_joint5"/>
-        <xacro:configure_joint name="fr3_joint6"/>
-        <xacro:configure_joint name="fr3_joint7"/>
+        <xacro:configure_joint name="fr3_joint1" ip="0.0"/>
+        <xacro:configure_joint name="fr3_joint2" ip="${-pi/4}"/>   <xacro:configure_joint name="fr3_joint3" ip="0.0"/>
+        <xacro:configure_joint name="fr3_joint4" ip="${-3*pi/4}"/> <xacro:configure_joint name="fr3_joint5" ip="0.0"/>
+        <xacro:configure_joint name="fr3_joint6" ip="${pi/2}"/>    <xacro:configure_joint name="fr3_joint7" ip="${pi/4}"/>    ```
         <joint name="fr3_finger_joint1">
             <command_interface name="position"/>
@@ -49,5 +50,4 @@
         </joint>
         <joint name="fr3_finger_joint2">
-            <!-- <command_interface name="position"/> -->
             <state_interface name="position"/>
             <state_interface name="velocity"/>
